File: Hardware/PCB/ao_audio_mixer/ao_audio_mixer.kicad_pcb (KiCad board)
At the start: 2 copper layers, 166 x 116 mm, 40 parts, among them J1 2 Pin Molex Header, J2 2 Pin Molex Header, J3 2 Pin Molex Header, J4 Synth_power_2x5, J5 Conn_01x06, J6 Conn_01x06, J7 2 Pin Molex Header, J8 2 Pin Molex Header, U1 TL072

Commit message: Final tweaks before fabbing
Other:
- board text added: "Main board"
- board text added: "Pots board"

Commit message: submodules
Parts:
- moved GRAF3 4.00 mm to (99.0, 54.0)
Other:
- board text added: "https://github.com/holmesrichards/audiomixer"

Commit message: board mount jacks
Parts:
- removed C1, C2, C3: 1uF, ao_tht:C_Rect_L7.2mm_W7.2mm_P5.00mm_FKS2_FKP2_MKS2_MKP2
- removed C4, C5: 10uF, ao_tht:CP_Radial_D6.3mm_P2.50mm
- removed C6, C7: 100nF, ao_tht:C_Disc_D3.0mm_W1.6mm_P2.50mm
- removed D1, D2: 1N5817, ao_tht:D_DO-41_SOD81_P7.62mm_Horizontal
- removed GRAF2: AO Logo, ao_tht:analogoutput
- removed GRAF3: CC0 Logo, ao_tht:CC0_logo
- removed H1, H2, H3, H4: MountingHole, ao_tht:MountingHole_3.2mm_M3
- removed the J4 at (112.4, 95.0)
- removed J7, J8: 2 Pin Molex Header, ao_tht:Molex_KK-254_AE-6410-02A_1x02_P2.54mm_Vertical
- removed R1, R2, R3: 100k, ao_tht:R_Axial_DIN0207_L6.3mm_D2.5mm_P10.16mm_Horizontal
- removed R4, R5: 10k, ao_tht:R_Axial_DIN0207_L6.3mm_D2.5mm_P10.16mm_Horizontal
- removed R6, R7: 1k, ao_tht:R_Axial_DIN0207_L6.3mm_D2.5mm_P10.16mm_Horizontal
- removed U1: TL072, ao_tht:DIP-8_W7.62mm_Socket_LongPads
- added J5: AudioJack2, ao_tht:Jack_6.35mm_PJ_629HAN, F.Cu at (190.0, 194.0)
- J1, J2, J3: value 2 Pin Molex Header -> AudioJack2; footprint ao_tht:Molex_KK-254_AE-6410-02A_1x02_P2.54mm_Vertical -> ao_tht:Jack_6.35mm_PJ_629HAN; moved to F.Cu
- J4: renamed from J5; value Conn_01x06 -> Conn_01x08; footprint Connector_PinSocket_2.54mm:PinSocket_1x06_P2.54mm_Vertical -> Connector_PinSocket_2.54mm:PinSocket_1x08_P2.54mm_Vertical
- J6: value Conn_01x06 -> AudioJack2; footprint Connector_PinHeader_2.54mm:PinHeader_1x06_P2.54mm_Vertical -> ao_tht:Jack_6.35mm_PJ_629HAN
- moved J6 143.0 mm to (212.5, 194.0), turned to 270 degrees
- moved GRAF1 66.6 mm to (190.0, 119.0)
- moved J3 32.6 mm to (212.5, 169.0), turned to 270 degrees
- moved J2 25.5 mm to (190.0, 169.0), turned to 270 degrees
- moved J1 23.2 mm to (167.5, 169.0), turned to 270 degrees
Routing:
- net Net-(J6-Pad5): track 102.1 -> 0.00 mm
- net Net-(J6-Pad6): track 96.1 -> 0.00 mm
- net /OUT2: track 90.0 -> 0.00 mm
- net /OUT1: track 84.0 -> 0.00 mm
- net /OUT1P: track 0.00 -> 75.1 mm
- net /OUT2P: track 0.00 -> 64.9 mm
- net -12V: track 54.2 -> 0.00 mm
- net +12V: track 41.3 -> 0.00 mm
- net Net-(R5-Pad1): track 30.1 -> 0.00 mm
- net Net-(C1-Pad2): track 29.1 -> 0.00 mm
- net Net-(C3-Pad2): track 28.1 -> 0.00 mm
- net /IN3: track 130.0 -> 155.3 mm
- net Net-(C2-Pad2): track 24.1 -> 0.00 mm
- net /IN2: track 106.6 -> 126.5 mm
- net /-12_IN: track 16.3 -> 0.00 mm
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- removed copper zone on B.Cu, net GND
- removed copper zone on F.Cu, net GND
Other:
- board size 166 x 116 mm -> 66 x 170 mm
- board text added: "Panel components board"
- board text removed: "Main board"
- board text removed: "OUT1"
- board text removed: "OUT2"
- board text removed: "Pots board"
- board text removed: "Rich Holmes CC0 1.0 April 2021"
- board text removed: "https://github.com/holmesrichards/audiomixer"

Commit message: Restore deleted board
Parts:
- added C1: 1uF, ao_tht:C_Rect_L7.2mm_W7.2mm_P5.00mm_FKS2_FKP2_MKS2_MKP2, B.Cu at (76.7, 112.8)
- added C2: 1uF, ao_tht:C_Rect_L7.2mm_W7.2mm_P5.00mm_FKS2_FKP2_MKS2_MKP2, B.Cu at (91.9, 112.8)
- added C3: 1uF, ao_tht:C_Rect_L7.2mm_W7.2mm_P5.00mm_FKS2_FKP2_MKS2_MKP2, B.Cu at (107.2, 112.8)
- added C4: 10uF, ao_tht:CP_Radial_D6.3mm_P2.50mm, B.Cu at (124.9, 64.6)
- added C5: 10uF, ao_tht:CP_Radial_D6.3mm_P2.50mm, B.Cu at (127.5, 115.4)
- added C6: 100nF, ao_tht:C_Disc_D3.0mm_W1.6mm_P2.50mm, B.Cu at (94.5, 74.7)
- added C7: 100nF, ao_tht:C_Disc_D3.0mm_W1.6mm_P2.50mm, B.Cu at (86.8, 95.0)
- added D1: 1N5817, ao_tht:D_DO-41_SOD81_P7.62mm_Horizontal, B.Cu at (119.9, 72.2)
- added D2: 1N5817, ao_tht:D_DO-41_SOD81_P7.62mm_Horizontal, B.Cu at (127.5, 107.7)
- added GRAF1: Panel holes, ao_audio_mixer:ao_audio_mixer_panel_slide_holes, F.Cu at (-76.1, 26.0)
- added GRAF2: AO Logo, ao_tht:analogoutput, B.Cu at (83.0, 46.0)
- added GRAF3: CC0 Logo, ao_tht:CC0_logo, B.Cu at (109.0, 54.0)
- added H1: MountingHole, ao_tht:MountingHole_3.2mm_M3, B.Cu at (70.0, 39.0)
- added H2: MountingHole, ao_tht:MountingHole_3.2mm_M3, B.Cu at (130.0, 39.0)
- added H3: MountingHole, ao_tht:MountingHole_3.2mm_M3, F.Cu at (70.0, 144.0)
- added H4: MountingHole, ao_tht:MountingHole_3.2mm_M3, F.Cu at (130.0, 144.0)
- added J7: Conn_01x08, Connector_PinHeader_2.54mm:PinHeader_1x08_P2.54mm_Vertical, F.Cu at (91.9, 135.7)
- added J8: Synth_power_2x5, ao_tht:Power_Header, B.Cu at (122.4, 95.0)
- added R1: 100k, ao_tht:R_Axial_DIN0207_L6.3mm_D2.5mm_P10.16mm_Horizontal, B.Cu at (76.7, 92.5)
- added R2: 100k, ao_tht:R_Axial_DIN0207_L6.3mm_D2.5mm_P10.16mm_Horizontal, B.Cu at (91.9, 92.5)
- added R3: 100k, ao_tht:R_Axial_DIN0207_L6.3mm_D2.5mm_P10.16mm_Horizontal, B.Cu at (107.2, 92.5)
- added R4: 10k, ao_tht:R_Axial_DIN0207_L6.3mm_D2.5mm_P10.16mm_Horizontal, B.Cu at (84.3, 74.7)
- added R5: 10k, ao_tht:R_Axial_DIN0207_L6.3mm_D2.5mm_P10.16mm_Horizontal, B.Cu at (89.4, 64.6)
- added R6: 1k, ao_tht:R_Axial_DIN0207_L6.3mm_D2.5mm_P10.16mm_Horizontal, B.Cu at (104.6, 74.7)
- added R7: 1k, ao_tht:R_Axial_DIN0207_L6.3mm_D2.5mm_P10.16mm_Horizontal, B.Cu at (99.5, 74.7)
- added U1: TL072, ao_tht:DIP-8_W7.62mm_Socket_LongPads, B.Cu at (94.5, 87.4)
Routing:
- net Net-(J7-Pad5): track 0.00 -> 96.7 mm
- net Net-(J7-Pad6): track 0.00 -> 90.6 mm
- net OUT1: track 0.00 -> 72.4 mm
- net OUT2: track 0.00 -> 69.4 mm
- net -12V: track 0.00 -> 54.2 mm
- net +12V: track 0.00 -> 41.3 mm
- net Net-(R5-Pad1): track 0.00 -> 30.1 mm
- net Net-(C1-Pad2): track 0.00 -> 29.1 mm
- net Net-(C3-Pad2): track 0.00 -> 28.1 mm
- net Net-(C2-Pad2): track 0.00 -> 24.1 mm
- net /-12_IN: track 0.00 -> 16.3 mm
- net /+12_IN: track 0.00 -> 16.3 mm
- net Net-(R4-Pad1): track 0.00 -> 10.2 mm
- net Net-(C3-Pad1): track 0.00 -> 10.2 mm
- net Net-(C2-Pad1): track 0.00 -> 10.2 mm
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- added copper zone on B.Cu, net GND
- added copper zone on F.Cu, net GND
Other:
- board size 66 x 170 mm -> 156 x 170 mm
- board text added: "Main board"
- board text added: "Rich Holmes CC0 1.0 April 2021"
- board text added: "https://github.com/holmesrichards/audiomixer"

Commit message: Documentation and final fixes before release
Other:
- board text removed: "IN1"
- board text removed: "IN2"
- board text removed: "IN3"
